File: KAT pcb/KAT pcb.kicad_sch (KiCad schematic)
At the start: 2 parts, among them U1 ATmega32U4-A

Commit message: Basic schematic
Parts:
- added C1: C_Small, symbol Device:C_Small
- added R2, R3: 22, symbol Device:R_Small
- R1: value R_Small -> 10k
Connections:
- net GND: now also C1.2
- net at U1.3 (D-): now also R3.1
- net at U1.4 (D+): now also R2.1
- net at U1.6 (UCAP): now also C1.1
